File: HARDWARE/CANbus-BLEHID/CANbus-BLEHID.kicad_pcb (KiCad board)
At the start: 2 copper layers, 63 x 45 mm, 60 parts, among them J1 AC300V-04P-5.0, J2 UART, SW1 SW_Push_Dual, U1 MCP2515-xST, U2 TLE7250V, U3 MP2315GJ-Z, U4 MIC5504-3.3YM5, U5 nRF51822-QFAC, Y1 16M, Y2 16M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

Commit message: PCB production and assembly files
Parts:
- REF**: value WEEE-Logo_4.2x6mm_SilkScreen -> WEEE
