File: HARDWARE/CANbus-BLEHID/CANbus-BLEHID.sch (KiCad schematic (older format))
At the start: 59 parts, among them J1 AC300V-04P-5.0, J2 UART, SW1 SW_Push_Dual, U1 MCP2515-xST, U2 TLE7250V, U3 MP2315GJ-Z, U4 MIC5504-3.3YM5, U5 nRF51822-QFAC, Y1 16M, Y2 16M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

Commit message: PCB production and assembly files
Parts:
- J1: footprint TerminalBlock:TerminalBlock_Altech_AK300-4_P5.00mm -> TerminalBlock_Phoenix:TerminalBlock_Phoenix_MKDS-1,5-4_1x04_P5.00mm_Horizontal
Changed lines of the file:
@@
 F 0 "J1" H 600 1450 50  0000 C CNN
 F 1 "AC300V-04P-5.0" H 350 1550 50  0000 C CNN
-F 2 "TerminalBlock:TerminalBlock_Altech_AK300-4_P5.00mm" H 600 1250 50  0001 C CNN
+F 2 "TerminalBlock_Phoenix:TerminalBlock_Phoenix_MKDS-1,5-4_1x04_P5.00mm_Horizontal" H 600 1250 50  0001 C CNN
 F 3 "https://www.tme.eu/pl/details/tb-5.0-p-4p1_gy/listwy-zaciskowe-do-druku/ninigi/ac300v-04p-5-0-gray/" H 600 1250 50  0001 C CNN
 	1    600  1250
